File: hardware/air-quality.kicad_pcb (KiCad board)
At the start: 2 copper layers, 20 x 25 mm, 26 parts, among them P101 CON-SENSOR2, P102 DEBUG, P103 BOOT, U1 BME680, U103 DRILL, U104 DRILL, U105 DRILL, U106 DRILL, U2 XMC1XXX48

Commit message: Change capacitor footprint(s) to C0402F
Parts:
- C1, C103, C104, C105, C2, C3: footprint C0603F -> kicad-libraries:C0603F
- C101: footprint C0805 -> kicad-libraries:C0805
- C102: footprint C0402E -> kicad-libraries:C0402F
- D101: footprint D0603E -> kicad-libraries:D0603E
- P101: footprint CON-SENSOR2 -> kicad-libraries:CON-SENSOR2
- R101: footprint R0603F -> kicad-libraries:R0603F
- RP101: footprint 4X0402 -> kicad-libraries:4X0402
- U103, U104, U105, U106: footprint DRILL_NP -> kicad-libraries:DRILL_NP
- moved C102 0.15 mm to (148.7, 136.8)
Connections:
- P101 pad 1: (no net) -> +5V
- U2 pad 1: (no net) -> Net-(U2-Pad1)
- U2 pad 10: (no net) -> Net-(U2-Pad10)
- U2 pad 11: (no net) -> Net-(U2-Pad11)
- U2 pad 12: (no net) -> Net-(U2-Pad12)
- U2 pad 14: (no net) -> Net-(U2-Pad14)
- U2 pad 15: (no net) -> Net-(U2-Pad15)
- U2 pad 16: (no net) -> Net-(U2-Pad16)
- U2 pad 2: (no net) -> Net-(U2-Pad2)
- U2 pad 20: (no net) -> Net-(U2-Pad20)
- U2 pad 21: (no net) -> Net-(U2-Pad21)
- U2 pad 22: (no net) -> Net-(U2-Pad22)
- U2 pad 23: (no net) -> Net-(U2-Pad23)
- U2 pad 24: (no net) -> Net-(U2-Pad24)
- U2 pad 25: (no net) -> Net-(U2-Pad25)
- U2 pad 26: (no net) -> Net-(U2-Pad26)
- U2 pad 28: (no net) -> Net-(U2-Pad28)
- U2 pad 29: (no net) -> Net-(U2-Pad29)
- U2 pad 30: (no net) -> Net-(U2-Pad30)
- U2 pad 31: (no net) -> Net-(U2-Pad31)
- U2 pad 32: (no net) -> Net-(U2-Pad32)
- U2 pad 34: (no net) -> Net-(U2-Pad34)
- U2 pad 4: (no net) -> Net-(U2-Pad4)
- U2 pad 41: (no net) -> Net-(U2-Pad41)
- U2 pad 42: (no net) -> Net-(U2-Pad42)
- U2 pad 43: (no net) -> Net-(U2-Pad43)
- U2 pad 47: (no net) -> Net-(U2-Pad47)
- U2 pad 48: (no net) -> Net-(U2-Pad48)
- U2 pad 5: (no net) -> Net-(U2-Pad5)
- U2 pad 6: (no net) -> Net-(U2-Pad6)
- U2 pad 8: (no net) -> Net-(U2-Pad8)
- U2 pad 9: (no net) -> Net-(U2-Pad9)
