File: hardware/air-quality.kicad_pcb (KiCad board)
At the start: 2 copper layers, 20 x 25 mm, 26 parts, among them P101 CON-SENSOR2, P102 DEBUG, P103 BOOT, U1 BME680, U103 DRILL, U104 DRILL, U105 DRILL, U106 DRILL, U2 XMC1XXX48

Commit message: specify processor
Parts:
- U2: value XMC1XXX48 -> XMC14XX48
Changed lines of the file:
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@@
-(kicad_pcb (version 4) (host pcbnew 4.0.2+dfsg1-stable)
+(kicad_pcb (version 4) (host pcbnew 4.0.7-e2-6376~61~ubuntu18.04.1)
   (general
     (links 50)
     (no_connects 0)
-    (area 134.244999 127.644999 275.56786 157.715)
+    (area 134.244999 127.644999 275.49286 158.115)
     (thickness 1.6)
     (drawings 12)
@@
       (effects (font (size 0.29972 0.29972) (thickness 0.0762)))
     )
-    (fp_text value XMC1XXX48 (at 0 -0.7 135) (layer F.SilkS)
-      (effects (font (size 0.29972 0.29972) (thickness 0.0762)))
+    (fp_text value XMC14XX48 (at 0 -0.7 135) (layer F.SilkS)
+      (effects (font (size 0.29972 0.29972) (thickness 0.07493)))
     )
     (fp_circle (center -2.5 2.6) (end -2.4 2.8) (layer F.Fab) (width 0.05))
