File: hardware/air-quality.kicad_pcb (KiCad board)
At the start: 2 copper layers, 20 x 25 mm, 26 parts, among them P101 CON-SENSOR2, P102 DEBUG, P103 BOOT, U1 BME680, U103 DRILL, U104 DRILL, U105 DRILL, U106 DRILL, U2 XMC14XX48

Commit message: fixed libary, added sym-lib-table, changed processor to XMC1404
Parts:
- U2: value XMC14XX48 -> XMC1404
Changed lines of the file:
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@@
       (effects (font (size 0.29972 0.29972) (thickness 0.0762)))
     )
-    (fp_text value XMC14XX48 (at 0 -0.7 135) (layer F.SilkS)
+    (fp_text value XMC1404 (at 0 -0.7 135) (layer F.SilkS)
       (effects (font (size 0.29972 0.29972) (thickness 0.07493)))
     )

Commit message: update to new kicad version
Other:
- net class Default removed
